File: Heathkit Curve Tracer Mods.kicad_sch (KiCad schematic)
At the start: 13 parts, among them J1 Switch, J2 IC6 Jumper, J3 +15, U1 74LS42, U2 74LVC1G04, U3 74LS90, U4 LM7805_TO220

Commit message: update
Connections:
- net GND: now also J2.6 (Pin_6)
Changed lines of the file:
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@@
+	)
+	(junction
+		(at 198.12 85.09)
+		(diameter 0)
+		(color 0 0 0 0)
 	)
 	(junction
@@
 	(wire
 		(pts
-			(xy 198.12 82.55) (xy 198.12 74.93)
+			(xy 198.12 86.36) (xy 198.12 85.09)
 		)
 		(stroke
@@
 	(wire
 		(pts
+			(xy 198.12 85.09) (xy 198.12 74.93)
+		)
+		(stroke
+			(width 0)
+			(type default)
+		)
+	)
+	(wire
+		(pts
 			(xy 241.3 43.18) (xy 241.3 38.1)
 		)
@@
 	(wire
 		(pts
+			(xy 177.8 85.09) (xy 198.12 85.09)
+		)
+		(stroke
+			(width 0)
+			(type default)
+		)
+	)
+	(wire
+		(pts
 			(xy 176.53 132.08) (xy 176.53 138.43)
 		)
@@
 	(wire
 		(pts
+			(xy 177.8 77.47) (xy 177.8 85.09)
+		)
+		(stroke
+			(width 0)
+			(type default)
+		)
+	)
+	(wire
+		(pts
 			(xy 74.93 90.17) (xy 106.68 90.17)
 		)
@@
 		(pts
 			(xy 157.48 43.18) (xy 128.27 43.18)
+		)
+		(stroke
+			(width 0)
+			(type default)
+		)
+	)
+	(wire
+		(pts
+			(xy 182.88 77.47) (xy 177.8 77.47)
 		)
 		(stroke
@@
 	(symbol
 		(lib_id "power:GND")
-		(at 198.12 82.55 0)
+		(at 198.12 86.36 0)
 		(unit 1)
 		(body_style 1)
@@
 		(dnp no)
 		(property "Reference" "#PWR013"
-			(at 198.12 88.9 0)
+			(at 198.12 92.71 0)
 			(hide yes)
 			(show_name no)
@@
 		)
 		(property "Value" "GND"
+			(at 198.12 90.17 0)
+			(show_name no)
+			(do_not_autoplace no)
+			(effects
+				(font
+					(size 1.27 1.27)
+				)
+			)
+		)
+		(property "Footprint" ""
 			(at 198.12 86.36 0)
-			(show_name no)
-			(do_not_autoplace no)
-			(effects
-				(font
-					(size 1.27 1.27)
-				)
-			)
-		)
-		(property "Footprint" ""
-			(at 198.12 82.55 0)
 			(hide yes)
 			(show_name no)
@@
 		)
 		(property "Datasheet" ""
-			(at 198.12 82.55 0)
+			(at 198.12 86.36 0)
 			(hide yes)
 			(show_name no)
@@
 		)
 		(property "Description" "Power symbol creates a global label with name \"GND\" , ground"
-			(at 198.12 82.55 0)
-			(hide yes)
-			(show_name no)
+			(at 198.12 86.36 0)
+			(hide yes)
+			(show_name no)
